Commit message: Align go2 description with Unitree's go2.urdf
Masses, inertias, joint origins, foot radius and the IMU mount (-0.02557, 0, 0.04232) now match
the Unitree URDF the Isaac training asset is built from (16.087 kg). The calf collision stays a
single box because the Gazebo foot contact sensors reference its lumped collision name.
robots/go2.urdf regenerated from the xacro.

File: robots/go2.urdf (robot description, URDF)
Before this commit: robot go2, 19 links, 18 joints
Links:
- added link head_lower, mass 0.001; collision sphere radius=0.047
- added link head_upper, mass 0.001; collision cylinder length=0.09 radius=0.05
- added link lf_haa_rotor, mass 0.089
- added link lf_hfe_rotor, mass 0.089
- added link lf_kfe_rotor, mass 0.089
- added link lh_haa_rotor, mass 0.089
- added link lh_hfe_rotor, mass 0.089
- added link lh_kfe_rotor, mass 0.089
- added link rf_haa_rotor, mass 0.089
- added link rf_hfe_rotor, mass 0.089
- added link rf_kfe_rotor, mass 0.089
- added link rh_haa_rotor, mass 0.089
- added link rh_hfe_rotor, mass 0.089
- added link rh_kfe_rotor, mass 0.089
- link imu_link: mass 0.001 -> 0; geometry 
- link lf_foot: mass 0.06 -> 0.04; geometry collision sphere radius=0.022; visual sphere radius=0.011999999999999999
- link lh_foot: mass 0.06 -> 0.04; geometry collision sphere radius=0.022; visual sphere radius=0.011999999999999999
- link rf_foot: mass 0.06 -> 0.04; geometry collision sphere radius=0.022; visual sphere radius=0.011999999999999999
- link rh_foot: mass 0.06 -> 0.04; geometry collision sphere radius=0.022; visual sphere radius=0.011999999999999999
Joints:
- added joint head_lower_joint: type fixed, parent head_upper, child head_lower, origin xyz=0.008 0 -0.07 rpy=0 0 0
- added joint head_upper_joint: type fixed, parent trunk, child head_upper, origin xyz=0.285 0 0.01 rpy=0 0 0
- added joint lf_haa_rotor_joint: type fixed, parent trunk, child lf_haa_rotor, origin xyz=0.11215 0.04675 0 rpy=0 0 0
- added joint lf_hfe_rotor_joint: type fixed, parent lf_hip, child lf_hfe_rotor, origin xyz=0 -0.00015 0 rpy=0 0 0
- added joint lf_kfe_rotor_joint: type fixed, parent lf_upperleg, child lf_kfe_rotor, origin xyz=0 -0.03235 0 rpy=0 0 0
- added joint lh_haa_rotor_joint: type fixed, parent trunk, child lh_haa_rotor, origin xyz=-0.11215 0.04675 0 rpy=0 0 0
- added joint lh_hfe_rotor_joint: type fixed, parent lh_hip, child lh_hfe_rotor, origin xyz=0 -0.00015 0 rpy=0 0 0
- added joint lh_kfe_rotor_joint: type fixed, parent lh_upperleg, child lh_kfe_rotor, origin xyz=0 -0.03235 0 rpy=0 0 0
- added joint rf_haa_rotor_joint: type fixed, parent trunk, child rf_haa_rotor, origin xyz=0.11215 -0.04675 0 rpy=0 0 0
- added joint rf_hfe_rotor_joint: type fixed, parent rf_hip, child rf_hfe_rotor, origin xyz=0 0.00015 0 rpy=0 0 0
- added joint rf_kfe_rotor_joint: type fixed, parent rf_upperleg, child rf_kfe_rotor, origin xyz=0 0.03235 0 rpy=0 0 0
- added joint rh_haa_rotor_joint: type fixed, parent trunk, child rh_haa_rotor, origin xyz=-0.11215 -0.04675 0 rpy=0 0 0
- added joint rh_hfe_rotor_joint: type fixed, parent rh_hip, child rh_hfe_rotor, origin xyz=0 0.00015 0 rpy=0 0 0
- added joint rh_kfe_rotor_joint: type fixed, parent rh_upperleg, child rh_kfe_rotor, origin xyz=0 0.03235 0 rpy=0 0 0
- joint imu_joint: origin xyz=-0.01592 -0.06659 -0.00617 rpy=0 0 0 -> xyz=-0.02557 0 0.04232 rpy=0 0 0
- joint lf_kfe_joint: limit lower=-2.7227 upper=-0.83776 effort=35.55 velocity=20.06 -> lower=-2.7227 upper=-0.83776 effort=45.43 velocity=15.7
- joint lh_hfe_joint: limit lower=-1.5708 upper=3.4907 effort=23.7 velocity=30.1 -> lower=-0.5236 upper=4.5379 effort=23.7 velocity=30.1
- joint lh_kfe_joint: limit lower=-2.7227 upper=-0.83776 effort=35.55 velocity=20.06 -> lower=-2.7227 upper=-0.83776 effort=45.43 velocity=15.7
- joint rf_kfe_joint: limit lower=-2.7227 upper=-0.83776 effort=35.55 velocity=20.06 -> lower=-2.7227 upper=-0.83776 effort=45.43 velocity=15.7
- joint rh_hfe_joint: limit lower=-1.5708 upper=3.4907 effort=23.7 velocity=30.1 -> lower=-0.5236 upper=4.5379 effort=23.7 velocity=30.1
- joint rh_kfe_joint: limit lower=-2.7227 upper=-0.83776 effort=35.55 velocity=20.06 -> lower=-2.7227 upper=-0.83776 effort=45.43 velocity=15.7

File: robots/go2.urdf.xacro (robot description, xacro)
@@ -37,26 +37,53 @@
         </inertial>
     </link>
+    <!-- Unitree's go2.urdf placement, i.e. where the real robot's IMU is -->
     <joint name="imu_joint" type="fixed">
         <parent link="trunk"/>
         <child link="imu_link"/>
-        <origin rpy="0 0 0" xyz="-0.01592 -0.06659 -0.00617"/>
+        <origin rpy="0 0 0" xyz="-0.02557 0 0.04232"/>
     </joint>
+    <!-- Identical to Unitree's imu_link: a massless frame with no geometry. The Gazebo IMU sensor
+         (gazebo/gazebo.xacro) is attached here with zero extra offset. -->
     <link name="imu_link">
         <inertial>
+            <origin rpy="0 0 0" xyz="0 0 0"/>
+            <mass value="0"/>
+            <inertia ixx="0" ixy="0" ixz="0" iyy="0" iyz="0" izz="0"/>
+        </inertial>
+    </link>
+    <!-- Head shells (Unitree's head_upper / head_lower): collision only, negligible mass -->
+    <joint name="head_upper_joint" type="fixed">
+        <origin rpy="0 0 0" xyz="0.285 0 0.01"/>
+        <parent link="trunk"/>
+        <child link="head_upper"/>
+    </joint>
+    <link name="head_upper">
+        <inertial>
+            <origin rpy="0 0 0" xyz="0 0 0"/>
             <mass value="0.001"/>
-            <origin rpy="0 0 0" xyz="0 0 0"/>
-            <inertia ixx="0.0001" ixy="0" ixz="0" iyy="0.0001" iyz="0" izz="0.0001"/>
+            <inertia ixx="9.6e-06" ixy="0" ixz="0" iyy="9.6e-06" iyz="0" izz="9.6e-06"/>
         </inertial>
-        <visual>
-            <origin rpy="0 0 0" xyz="0 0 0"/>
-            <geometry>
-                <box size="0.001 0.001 0.001"/>
-            </geometry>
-            <!-- <material name="red"/> -->
-        </visual>
         <collision>
             <origin rpy="0 0 0" xyz="0 0 0"/>
             <geometry>
-                <box size=".001 .001 .001"/>
+                <cylinder radius="0.05" length="0.09"/>
+            </geometry>
+        </collision>
+    </link>
+    <joint name="head_lower_joint" type="fixed">
+        <origin rpy="0 0 0" xyz="0.008 0 -0.07"/>
+        <parent link="head_upper"/>
+        <child link="head_lower"/>
+    </joint>
+    <link name="head_lower">
+        <inertial>
+            <origin rpy="0 0 0" xyz="0 0 0"/>
+            <mass value="0.001"/>
+            <inertia ixx="9.6e-06" ixy="0" ixz="0" iyy="9.6e-06" iyz="0" izz="9.6e-06"/>
+        </inertial>
+        <collision>
+            <origin rpy="0 0 0" xyz="0 0 0"/>
+            <geometry>
+                <sphere radius="0.047"/>
             </geometry>
         </collision>

File: urdfs/const.xacro (robot description, xacro)
@@ -1,5 +1,7 @@
 <?xml version="1.0"?>
 <robot xmlns:xacro="http://www.ros.org/wiki/xacro">
-    <!-- Constants for robot dimensions -->
+    <!-- Constants for robot dimensions.
+         Aligned with Unitree's go2.urdf (the one safe_rl trains on): joint limits, motor rotor
+         masses, foot, hip collision and IMU placement. Names stay locosim's. -->
     <xacro:property name="PI" value="3.1415926535897931"/>
     <xacro:property name="stick_mass" value="0.00001"/>
@@ -10,4 +12,6 @@
     <xacro:property name="hip_radius" value="0.046"/>
     <xacro:property name="hip_length" value="0.04"/>
+    <!-- lateral offset of the hip collision cylinder (Unitree: 0.08, not the 0.0955 joint offset) -->
+    <xacro:property name="hip_collision_offset" value="0.08"/>
     <xacro:property name="upperleg_shoulder_radius" value="0.041"/>
     <xacro:property name="upperleg_shoulder_length" value="0.032"/>
@@ -16,5 +20,7 @@
     <xacro:property name="lowerleg_width" value="0.016"/>
     <xacro:property name="lowerleg_height" value="0.016"/>
-    <xacro:property name="foot_radius" value="0.02"/>
+    <xacro:property name="foot_radius" value="0.022"/>
+    <!-- the foot sphere sits 2 mm behind the foot frame -->
+    <xacro:property name="foot_collision_offset_x" value="-0.002"/>
     <xacro:property name="stick_radius" value="0.01"/>
     <xacro:property name="stick_length" value="0.2"/>
@@ -47,10 +53,13 @@
     <xacro:property name="hfe_max" value="3.4907"/>
     <xacro:property name="hfe_min" value="-1.5708"/>
+    <!-- the hind thighs have a different range from the front ones -->
+    <xacro:property name="hfe_max_hind" value="4.5379"/>
+    <xacro:property name="hfe_min_hind" value="-0.5236"/>
     <xacro:property name="hfe_velocity_max" value="30.1"/>
     <xacro:property name="hfe_torque_max" value="23.7"/>
     <xacro:property name="kfe_max" value="-0.83776"/>
     <xacro:property name="kfe_min" value="-2.7227"/>
-    <xacro:property name="kfe_velocity_max" value="20.06"/>
-    <xacro:property name="kfe_torque_max" value="35.55"/>
+    <xacro:property name="kfe_velocity_max" value="15.70"/>
+    <xacro:property name="kfe_torque_max" value="45.43"/>
     <!-- dynamics inertial value -->
     <!-- trunk -->
@@ -99,4 +108,15 @@
     <xacro:property name="lowerleg_izz" value="3.29E-05"/>
     <!-- foot -->
-    <xacro:property name="foot_mass" value="0.06"/>
+    <xacro:property name="foot_mass" value="0.04"/>
+    <xacro:property name="foot_inertia" value="9.6e-06"/>
+    <!-- motor rotors, fixed to the body that carries each motor (Unitree's *_rotor links):
+         haa rotor on the trunk, hfe rotor on the hip, kfe rotor on the upper leg.
+         Offsets are for the left front leg; y flips with mirror, x with front_hind. -->
+    <xacro:property name="rotor_mass" value="0.089"/>
+    <xacro:property name="rotor_i_axis" value="0.000111842"/>
+    <xacro:property name="rotor_i_radial" value="0.000059647"/>
+    <xacro:property name="haa_rotor_offset_x" value="0.11215"/>
+    <xacro:property name="haa_rotor_offset_y" value="0.04675"/>
+    <xacro:property name="hfe_rotor_offset_y" value="-0.00015"/>
+    <xacro:property name="kfe_rotor_offset_y" value="-0.03235"/>
 </robot>

File: urdfs/leg.xacro (robot description, xacro)
@@ -49,5 +49,5 @@
             </visual>
             <collision>
-                <origin rpy="${PI/2.0} 0 0" xyz="0 ${hip_offset*mirror} 0"/>
+                <origin rpy="${PI/2.0} 0 0" xyz="0 ${hip_collision_offset*mirror} 0"/>
                 <geometry>
                     <cylinder length="${hip_length}" radius="${hip_radius}"/>
@@ -69,5 +69,10 @@
             <axis xyz="0 1 0"/>
             <dynamics damping="${damping}" friction="${friction}"/>
-            <limit effort="${hfe_torque_max}" velocity="${hfe_velocity_max}" lower="${hfe_min}" upper="${hfe_max}"/>
+            <xacro:if value="${front_hind_dae == True}">
+                <limit effort="${hfe_torque_max}" velocity="${hfe_velocity_max}" lower="${hfe_min}" upper="${hfe_max}"/>
+            </xacro:if>
+            <xacro:if value="${front_hind_dae == False}">
+                <limit effort="${hfe_torque_max}" velocity="${hfe_velocity_max}" lower="${hfe_min_hind}" upper="${hfe_max_hind}"/>
+            </xacro:if>
         </joint>
         <link name="${name}_upperleg">
@@ -122,9 +127,9 @@
             </collision>
             <inertial>
-                <origin rpy="0 0 0" xyz="${lowerleg_com_x} ${lowerleg_com_y} ${lowerleg_com_z}"/>
+                <origin rpy="0 0 0" xyz="${lowerleg_com_x} ${lowerleg_com_y*mirror} ${lowerleg_com_z}"/>
                 <mass value="${lowerleg_mass}"/>
                 <inertia
-                    ixx="${lowerleg_ixx}" ixy="${lowerleg_ixy}" ixz="${lowerleg_ixz}"
-                    iyy="${lowerleg_iyy}" iyz="${lowerleg_iyz}"
+                    ixx="${lowerleg_ixx}" ixy="${lowerleg_ixy*mirror}" ixz="${lowerleg_ixz}"
+                    iyy="${lowerleg_iyy}" iyz="${lowerleg_iyz*mirror}"
                     izz="${lowerleg_izz}"/>
             </inertial>
@@ -144,5 +149,5 @@
             </visual>
             <collision>
-                <origin rpy="0 0 0" xyz="0 0 0"/>
+                <origin rpy="0 0 0" xyz="${foot_collision_offset_x} 0 0"/>
                 <geometry>
                     <sphere radius="${foot_radius}"/>
@@ -152,7 +157,49 @@
                 <mass value="${foot_mass}"/>
                 <inertia
-                    ixx="${(2*foot_mass)/5.0*(foot_radius*foot_radius)}" ixy="0.0" ixz="0.0"
-                    iyy="${(2*foot_mass)/5.0*(foot_radius*foot_radius)}" iyz="0.0"
-                    izz="${(2*foot_mass)/5.0*(foot_radius*foot_radius)}"/>
+                    ixx="${foot_inertia}" ixy="0.0" ixz="0.0"
+                    iyy="${foot_inertia}" iyz="0.0"
+                    izz="${foot_inertia}"/>
+            </inertial>
+        </link>
+        <!-- Motor rotors: mass only (fixed joints, no collision), so they lump into the body that
+             carries each motor - which is also what Isaac does with Unitree's *_rotor links. No
+             collision on purpose: the foot contact sensors reference lumped collision indices. -->
+        <joint name="${name}_haa_rotor_joint" type="fixed">
+            <origin rpy="0 0 0" xyz="${haa_rotor_offset_x*front_hind} ${haa_rotor_offset_y*mirror} 0"/>
+            <parent link="trunk"/>
+            <child link="${name}_haa_rotor"/>
+        </joint>
+        <link name="${name}_haa_rotor">
+            <inertial>
+                <origin rpy="0 0 0" xyz="0 0 0"/>
+                <mass value="${rotor_mass}"/>
+                <inertia ixx="${rotor_i_axis}" ixy="0.0" ixz="0.0"
+                         iyy="${rotor_i_radial}" iyz="0.0" izz="${rotor_i_radial}"/>
+            </inertial>
+        </link>
+        <joint name="${name}_hfe_rotor_joint" type="fixed">
+            <origin rpy="0 0 0" xyz="0 ${hfe_rotor_offset_y*mirror} 0"/>
+            <parent link="${name}_hip"/>
+            <child link="${name}_hfe_rotor"/>
+        </joint>
+        <link name="${name}_hfe_rotor">
+            <inertial>
+                <origin rpy="0 0 0" xyz="0 0 0"/>
+                <mass value="${rotor_mass}"/>
+                <inertia ixx="${rotor_i_radial}" ixy="0.0" ixz="0.0"
+                         iyy="${rotor_i_axis}" iyz="0.0" izz="${rotor_i_radial}"/>
+            </inertial>
+        </link>
+        <joint name="${name}_kfe_rotor_joint" type="fixed">
+            <origin rpy="0 0 0" xyz="0 ${kfe_rotor_offset_y*mirror} 0"/>
+            <parent link="${name}_upperleg"/>
+            <child link="${name}_kfe_rotor"/>
+        </joint>
+        <link name="${name}_kfe_rotor">
+            <inertial>
+                <origin rpy="0 0 0" xyz="0 0 0"/>
+                <mass value="${rotor_mass}"/>
+                <inertia ixx="${rotor_i_radial}" ixy="0.0" ixz="0.0"
+                         iyy="${rotor_i_axis}" iyz="0.0" izz="${rotor_i_radial}"/>
             </inertial>
         </link>
