Commit message: Add the joint model of the RL policies
Joint friction, viscous damping and reflected rotor inertia from the PACE fit
of the real Go2 (safe_rl assets.py), averaged per joint type. The rotor inertia
is applied by locosim's libjoint_armature_plugin, since ODE has no armature.
Contact damping raised from 100 to 3000 N s/m: at 100 the feet bounce on
touchdown. robots/go2.urdf regenerated.

File: urdfs/const.xacro (robot description, xacro)
@@ -45,6 +45,13 @@
     <xacro:property name="lowerleg_offset_z" value="-0.213"/>
     <!-- joint limits -->
-    <xacro:property name="damping" value="0.0"/>
-    <xacro:property name="friction" value="0.0"/>
+    <!-- Joint model the RL policies are trained with: the PACE fit of the real robot
+         (safe_rl/assets.py, UNITREE_GO2_IDENTIFIED), averaged over the four legs per joint type.
+         Coulomb friction N m, viscous damping N m s/rad, reflected rotor inertia (armature) kg m^2,
+         applied by libjoint_armature_plugin (leg.xacro) since ODE has no armature. -->
+    <xacro:property name="joint_coulomb" value="${dict(haa=0.24, hfe=0.23, kfe=0.8)}"/>
+    <xacro:property name="joint_viscous" value="${dict(haa=0.25, hfe=0.22, kfe=0.29)}"/>
+    <xacro:property name="joint_armature" value="${dict(haa=0.02, hfe=0.023, kfe=0.037)}"/>
+    <!-- Contact damping, N s/m (leg.gazebo.xacro): at 100 the feet bounce on touchdown. -->
+    <xacro:property name="contact_kd" value="3000.0"/>
     <xacro:property name="haa_max" value="1.0472"/>
     <xacro:property name="haa_min" value="-1.0472"/>

File: urdfs/leg.gazebo.xacro (robot description, xacro)
@@ -23,5 +23,5 @@
 		<gazebo reference="${name}_upperleg">
 			<kp>1000000.0</kp>
-			<kd>100.0</kd>
+			<kd>${contact_kd}</kd>
 			<mu1>1.5</mu1>
 			<mu2>1.5</mu2>
@@ -32,5 +32,5 @@
 		<gazebo reference="${name}_lowerleg">
 			<kp>1000000.0</kp>
-			<kd>100.0</kd>
+			<kd>${contact_kd}</kd>
 			<mu1>1.0</mu1>
 			<mu2>1.0</mu2>
@@ -40,5 +40,5 @@
         <gazebo reference="${name}_foot">
             <kp>1000000.0</kp>
-            <kd>100.0</kd>
+            <kd>${contact_kd}</kd>
             <mu1>1.0</mu1>
             <mu2>1.0</mu2>

File: urdfs/leg.xacro (robot description, xacro)
@@ -21,5 +21,5 @@
             <child link="${name}_hip"/>
             <axis xyz="1 0 0"/>
-            <dynamics damping="${damping}" friction="${friction}"/>
+            <dynamics damping="${joint_viscous['haa']}" friction="${joint_coulomb['haa']}"/>
             <xacro:if value="${(mirror_dae == True)}">
                 <limit effort="${haa_torque_max}" velocity="${haa_velocity_max}" lower="${haa_min}" upper="${haa_max}"/>
@@ -68,5 +68,5 @@
             <child link="${name}_upperleg"/>
             <axis xyz="0 1 0"/>
-            <dynamics damping="${damping}" friction="${friction}"/>
+            <dynamics damping="${joint_viscous['hfe']}" friction="${joint_coulomb['hfe']}"/>
             <xacro:if value="${front_hind_dae == True}">
                 <limit effort="${hfe_torque_max}" velocity="${hfe_velocity_max}" lower="${hfe_min}" upper="${hfe_max}"/>
@@ -109,5 +109,5 @@
             <child link="${name}_lowerleg"/>
             <axis xyz="0 1 0"/>
-            <dynamics damping="${damping}" friction="${friction}"/>
+            <dynamics damping="${joint_viscous['kfe']}" friction="${joint_coulomb['kfe']}"/>
             <limit effort="${kfe_torque_max}" velocity="${kfe_velocity_max}" lower="${kfe_min}" upper="${kfe_max}"/>
         </joint>
@@ -206,4 +206,12 @@
         <xacro:leg_transmission name="${name}"/>
         <xacro:leg_gazebo name="${name}"/>
+        <!-- Reflected rotor inertia (const.xacro), built from gazebo_plugins/joint_armature_plugin -->
+        <gazebo>
+            <plugin name="joint_armature_${name}" filename="libjoint_armature_plugin.so">
+                <joint name="${name}_haa_joint">${joint_armature['haa']}</joint>
+                <joint name="${name}_hfe_joint">${joint_armature['hfe']}</joint>
+                <joint name="${name}_kfe_joint">${joint_armature['kfe']}</joint>
+            </plugin>
+        </gazebo>
     </xacro:macro>
 </robot>
